File: IRIS_KiCAD/IRIS_KiCAD.kicad_pcb (KiCad board)
At the start: 4 copper layers, 92.7 x 72.5 mm, 242 parts

Commit message: flipped XT60 connector to bottom + photorealistic renders
Parts:
- C1, C100, C103, C112, C113, C115, C116, C25, C27, C94: footprint LCSC_imported:C0603 -> ProPrj_IRI-easyedapro:C0603
- C10, C105, C106, C107, C108, C109, C11, C110, C114, C12, C2, C22, C24, C28, C29, C3, C31, C32, C39, C40, C41, C43, C51, C52, C53, C54, C60, C61, C62, C63, C66, C67, C69, C7, C71, C75, C76, C77, C78, C79, C8, C80, C81, C89, C9, C92, C93: footprint LCSC_imported:C0402 -> ProPrj_IRI-easyedapro:C0402
- C117, C118, C119, C120: footprint LCSC_imported:CAP-SMD_BD6.3-L6.6-W6.6-LS7.2-FD_3 -> ProPrj_IRI-easyedapro:CAP-SMD_BD6.3-L6.6-W6.6-LS7.2-FD_3
- C36, C37, C38, C4, C5, C55, C57, C58, C59, C6, C68, C70: footprint LCSC_imported:C0805 -> ProPrj_IRI-easyedapro:C0805
- C95: footprint LCSC_imported:C0402 -> ProPrj_IRI-easyedapro:C0402; moved to F.Cu
- C96: footprint LCSC_imported:C0805 -> ProPrj_IRI-easyedapro:C0805; moved to F.Cu
- C97, C98: footprint LCSC_imported:C0603 -> ProPrj_IRI-easyedapro:C0603; moved to F.Cu
- C99: footprint LCSC_imported:CAP-SMD_L3.2-W1.6-RD-C7171 -> ProPrj_IRI-easyedapro:CAP-SMD_L3.2-W1.6-RD-C7171
- CN1: footprint LCSC_imported:CONN-TH_XT60PW-M -> ProPrj_IRI-easyedapro:CONN-TH_XT60PW-M; moved to B.Cu
- FPC1: footprint LCSC_imported:FPC-SMD_24P-P0.50_FPC-05F-24PH20 -> ProPrj_IRI-easyedapro:FPC-SMD_24P-P0.50_FPC-05F-24PH20
- H1, H2, H3, H4, H5: footprint LCSC_imported:HDR-TH_4P-HX-PH254-01-04-Z-L11.5 -> ProPrj_IRI-easyedapro:HDR-TH_4P-HX-PH254-01-04-Z-L11.5
- L1, L2, L3, L4, L5: footprint LCSC_imported:L0402 -> ProPrj_IRI-easyedapro:L0402
- L6: footprint LCSC_imported:IND-SMD_L3.0-W3.0-1 -> ProPrj_IRI-easyedapro:IND-SMD_L3.0-W3.0-1; moved to F.Cu
- L7: footprint LCSC_imported:IND-SMD_L1.8-W1.0 -> ProPrj_IRI-easyedapro:IND-SMD_L1.8-W1.0
- L8: footprint LCSC_imported:ANT-TH_L18.0-W18.0_C9900026472 -> ProPrj_IRI-easyedapro:ANT-TH_L18.0-W18.0_C9900026472
- Q1, Q10, Q11, Q12, Q13, Q14, Q15, Q16, Q17, Q18, Q19, Q2, Q20, Q21, Q22, Q23, Q24, Q3, Q4, Q5, Q6, Q7, Q8, Q9: footprint LCSC_imported:TO-252-3_L6.6-W6.1-P4.57-LS9.9-BR-CW -> ProPrj_IRI-easyedapro:TO-252-3_L6.6-W6.1-P4.57-LS9.9-BR-CW
- R1, R10, R15, R16, R17, R19, R2, R20, R21, R22, R23, R24, R28, R29, R3, R30, R34, R36, R4, R41, R42, R43, R44, R45, R46, R47, R48, R49, R5, R57, R58, R59, R6, R60, R61, R62, R63, R64, R65, R66, R7, R74, R75, R76, R8, R81, R82, R9: footprint LCSC_imported:R0603 -> ProPrj_IRI-easyedapro:R0603
- R11, R12, R13, R14, R18, R25, R26, R27, R31, R32, R37, R38, R39, R40, R50, R51, R52, R53, R54, R55, R67, R68, R69, R70, R71, R72, R77, R78, R79, R80: footprint LCSC_imported:R0402 -> ProPrj_IRI-easyedapro:R0402
- R33: footprint LCSC_imported:R0603 -> ProPrj_IRI-easyedapro:R0603; moved to B.Cu
- U1, U10, U13, U14, U16, U17, U19, U20, U21, U22, U24, U7: footprint LCSC_imported:SOIC-8_L4.9-W3.9-P1.27-LS6.0-BL -> ProPrj_IRI-easyedapro:SOIC-8_L4.9-W3.9-P1.27-LS6.0-BL
- U11: footprint LCSC_imported:TSOT-23-6_L2.9-W1.6-P0.95-LS2.8-BL -> ProPrj_IRI-easyedapro:TSOT-23-6_L2.9-W1.6-P0.95-LS2.8-BL; moved to F.Cu
- U12, U35, U5, U6, U8: footprint LCSC_imported:SW-SMD_2P-L6.2-W2.5-LS9.4 -> ProPrj_IRI-easyedapro:SW-SMD_2P-L6.2-W2.5-LS9.4
- U15, U18, U23, U9: footprint LCSC_imported:LQFP-32_L7.0-W7.0-P0.80-LS9.0-BL -> ProPrj_IRI-easyedapro:LQFP-32_L7.0-W7.0-P0.80-LS9.0-BL
- U2: footprint LCSC_imported:LGA-14_L3.0-W2.5-P0.50-TL -> ProPrj_IRI-easyedapro:LGA-14_L3.0-W2.5-P0.50-TL
- U25: footprint LCSC_imported:SOT-223-4_L6.5-W3.5-P2.30-LS7.0-BR -> ProPrj_IRI-easyedapro:SOT-223-4_L6.5-W3.5-P2.30-LS7.0-BR
- U27: footprint LCSC_imported:GPSM-SMD_ATGM336H-TR -> ProPrj_IRI-easyedapro:GPSM-SMD_ATGM336H-TR
- U29: footprint LCSC_imported:SOT-23-3_L3.0-W1.6-P1.90-LS2.8-BR -> ProPrj_IRI-easyedapro:SOT-23-3_L3.0-W1.6-P1.90-LS2.8-BR
- U3: footprint LCSC_imported:LGA-8_L2.5-W2.0-P0.65_AMP6127 -> ProPrj_IRI-easyedapro:LGA-8_L2.5-W2.0-P0.65_AMP6127
- U30: footprint LCSC_imported:SOT-23-3_L2.9-W1.6-P1.90-LS2.8-BR -> ProPrj_IRI-easyedapro:SOT-23-3_L2.9-W1.6-P1.90-LS2.8-BR
- U31: footprint LCSC_imported:CRYSTAL-SMD_4P-L2.0-W1.6-BL -> ProPrj_IRI-easyedapro:CRYSTAL-SMD_4P-L2.0-W1.6-BL
- U32: footprint LCSC_imported:COMM-SMD_E01C-ML01SP4 -> ProPrj_IRI-easyedapro:COMM-SMD_E01C-ML01SP4
- U33: footprint LCSC_imported:LQFP-100_L14.0-W14.0-P0.50-LS16.0-BL -> ProPrj_IRI-easyedapro:LQFP-100_L14.0-W14.0-P0.50-LS16.0-BL
- U34: footprint LCSC_imported:SW-TH_SHOU-HAN_SS12D10G4 -> ProPrj_IRI-easyedapro:SW-TH_SHOU-HAN_SS12D10G4
- U4: footprint LCSC_imported:LGA-12_L2.0-W2.0-P0.50-BL -> ProPrj_IRI-easyedapro:LGA-12_L2.0-W2.0-P0.50-BL
- USB3: footprint LCSC_imported:USB-C-SMD_KH-TYPE-C-16P -> ProPrj_IRI-easyedapro:USB-C-SMD_KH-TYPE-C-16P
- moved C98 13.8 mm to (143.9, 126.0), turned to 180 degrees
- moved L6 10.6 mm to (142.4, 128.4), turned to 0 degrees
- moved C97 10.3 mm to (142.1, 131.1)
- moved R33 7.62 mm to (155.0, 124.6), turned to -90 degrees
- moved C95 6.63 mm to (140.2, 128.9), turned to 90 degrees
- moved U11 5.78 mm to (137.8, 129.3), turned to -90 degrees
- moved H2 2.62 mm to (147.3, 126.7), turned to 90 degrees
- moved CN1 1.26 mm to (138.2, 131.5), turned to -90 degrees
- moved C96 0.34 mm to (138.1, 132.0)
Routing:
- net $1N17368: track 15.4 -> 27.7 mm
- net $1N17546: track 6.84 -> 2.69 mm
- net BOOT0: track 9.72 -> 5.63 mm, vias 0 -> 1
- net GND: track 304.0 -> 301.3 mm, vias 169 -> 155
- net 7.4V_BATTERY: track 253.4 -> 255.6 mm, vias 182 -> 172
- net RADIO_TX: track 10.8 -> 8.56 mm, vias 1 -> 0
- net +5V: track 64.5 -> 66.0 mm
- net MOTOR3: track 80.5 -> 79.6 mm
