File: pcb/kicad/ProPrj_IRIS.kicad_sch (KiCad schematic)
At the start: 77 parts, among them CN1 XT60PW-M, SW5 LXW-4X3X2-SMD, U11 AP63205WU-7, U12 2.54-1P TPGT, U2 ICM-42688-P, U25 MIC39100-3.3WS-TR, U27 ATGM336H-5N31, U29 XC6206-1.2V, U3 BMP280, U30 XC6206-2.8V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

Commit message: corrected nrst decoupling capacitor - thanks to @kaipereira for the tip
Parts:
- removed ?: (no value), ProPrj_IRI-easyedapro:, symbol ProPrj_IRI-easyedapro:Drawing-Symbol_A4
- added ?: (no value), ProPrj_IRI-easyedapro:, symbol ProPrj_IRI-easyedapro:Drawing-Symbol_A4
- USB3: LCSC Part Name Type-C 母 卧贴 -> (none); Manufacturer kinghelm(金航标) -> (none); Manufacturer Part KH-TYPE-C-16P -> (none); Supplier LCSC -> (none); Supplier Part C709357 -> (none)
Connections:
- net GND: now also C121.2
- net VCC: no longer C121.1
- net at R76.2, SW5.2, U33.14 (NRST): now also C121.1; no longer C121.2
